Commit message: finish stand still, not complete interaction movement.

File: description/robots/g1/29dof_official.urdf (robot description, URDF)
Before this commit: robot g1_29dof_rev_1_0, 39 links, 38 joints
Links:
- link head_link: geometry collision mesh filename=/home/z/Desktop/PBHC/description/robots/g1/meshes/head_link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; visual mesh filename=/home/z/Desktop/PBHC/description/robots/g1/meshes/head_link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
- link left_ankle_pitch_link: geometry collision mesh filename=/home/z/Desktop/PBHC/description/robots/g1/meshes/left_ankl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; visual mesh filename=/home/z/Desktop/PBHC/description/robots/g1/meshes/left_ankl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
- link left_ankle_roll_link: geometry collision sphere radius=0.005; collision sphere radius=0.005
- link left_elbow_link: geometry collision mesh filename=/home/z/Desktop/PBHC/description/robots/g1/meshes/left_elbo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; visual mesh filename=/home/z/Desktop/PBHC/description/robots/g1/meshes/left_elbo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
- link left_hip_pitch_link: geometry collision mesh filename=/home/z/Desktop/PBHC/description/robots/g1/meshes/left_hip_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; visual mesh filename=/home/z/Desktop/PBHC/description/robots/g1/meshes/left_hip_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
- link left_hip_roll_link: geometry collision mesh filename=/home/z/Desktop/PBHC/description/robots/g1/meshes/left_hip_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; visual mesh filename=/home/z/Desktop/PBHC/description/robots/g1/meshes/left_hip_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
- link left_hip_yaw_link: geometry collision mesh filename=/home/z/Desktop/PBHC/description/robots/g1/meshes/left_hip_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; visual mesh filename=/home/z/Desktop/PBHC/description/robots/g1/meshes/left_hip_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
- link left_knee_link: geometry collision mesh filename=/home/z/Desktop/PBHC/description/robots/g1/meshes/left_knee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; visual mesh filename=/home/z/Desktop/PBHC/description/robots/g1/meshes/left_knee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
- link left_rubber_hand: geometry visual mesh filename=/home/z/Desktop/PBHC/description/robots/g1/meshes/left_rubb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
- link left_shoulder_pitch_link: geometry collision cylinder length=0.05 radius=0.03; visual mesh filename=/home/z/Desktop/PBHC/description/robots/g1/meshes/left_shou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
- link left_shoulder_roll_link: geometry collision cylinder length=0.03 radius=0.03; visual mesh filename=/home/z/Desktop/PBHC/description/robots/g1/meshes/left_shou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
- link left_shoulder_yaw_link: geometry collision mesh filename=/home/z/Desktop/PBHC/description/robots/g1/meshes/left_shou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; visual mesh filename=/home/z/Desktop/PBHC/description/robots/g1/meshes/left_shou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
- link left_wrist_pitch_link: geometry collision mesh filename=/home/z/Desktop/PBHC/description/robots/g1/meshes/left_wris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; visual mesh filename=/home/z/Desktop/PBHC/description/robots/g1/meshes/left_wris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
- link left_wrist_roll_link: geometry collision mesh filename=/home/z/Desktop/PBHC/description/robots/g1/meshes/left_wris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; visual mesh filename=/home/z/Desktop/PBHC/description/robots/g1/meshes/left_wris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
- link left_wrist_yaw_link: geometry collision mesh filename=/home/z/Desktop/PBHC/description/robots/g1/meshes/left_wris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; visual mesh filename=/home/z/Desktop/PBHC/description/robots/g1/meshes/left_wris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
- link logo_link: geometry collision mesh filename=/home/z/Desktop/PBHC/description/robots/g1/meshes/logo_link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; visual mesh filename=/home/z/Desktop/PBHC/description/robots/g1/meshes/logo_link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
- link pelvis: geometry visual mesh filename=/home/z/Desktop/PBHC/description/robots/g1/meshes/pelvis.STL
- link pelvis_contour_link: geometry collision mesh filename=/home/z/Desktop/PBHC/description/robots/g1/meshes/pelvis_co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; visual mesh filename=/home/z/Desktop/PBHC/description/robots/g1/meshes/pelvis_co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
- link right_ankle_pitch_link: geometry collision mesh filename=/home/z/Desktop/PBHC/description/robots/g1/meshes/right_ank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; visual mesh filename=/home/z/Desktop/PBHC/description/robots/g1/meshes/right_ank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
- link right_ankle_roll_link: geometry collision sphere radius=0.005; collision sphere radius=0.005
- link right_elbow_link: geometry collision mesh filename=/home/z/Desktop/PBHC/description/robots/g1/meshes/right_elb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; visual mesh filename=/home/z/Desktop/PBHC/description/robots/g1/meshes/right_elb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
- link right_hip_pitch_link: geometry collision mesh filename=/home/z/Desktop/PBHC/description/robots/g1/meshes/right_hip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; visual mesh filename=/home/z/Desktop/PBHC/description/robots/g1/meshes/right_hip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
- link right_hip_roll_link: geometry collision mesh filename=/home/z/Desktop/PBHC/description/robots/g1/meshes/right_hip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; visual mesh filename=/home/z/Desktop/PBHC/description/robots/g1/meshes/right_hip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
- link right_hip_yaw_link: geometry collision mesh filename=/home/z/Desktop/PBHC/description/robots/g1/meshes/right_hip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; visual mesh filename=/home/z/Desktop/PBHC/description/robots/g1/meshes/right_hip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
- link right_knee_link: geometry collision mesh filename=/home/z/Desktop/PBHC/description/robots/g1/meshes/right_kne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; visual mesh filename=/home/z/Desktop/PBHC/description/robots/g1/meshes/right_kne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
- link right_rubber_hand: geometry visual mesh filename=/home/z/Desktop/PBHC/description/robots/g1/meshes/right_rub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
- link right_shoulder_pitch_link: geometry collision cylinder length=0.05 radius=0.03; visual mesh filename=/home/z/Desktop/PBHC/description/robots/g1/meshes/right_sho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
- link right_shoulder_roll_link: geometry collision cylinder length=0.03 radius=0.03; visual mesh filename=/home/z/Desktop/PBHC/description/robots/g1/meshes/right_sho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
- link right_shoulder_yaw_link: geometry collision mesh filename=/home/z/Desktop/PBHC/description/robots/g1/meshes/right_sho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; visual mesh filename=/home/z/Desktop/PBHC/description/robots/g1/meshes/right_sho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
- link right_wrist_pitch_link: geometry collision mesh filename=/home/z/Desktop/PBHC/description/robots/g1/meshes/right_wri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; visual mesh filename=/home/z/Desktop/PBHC/description/robots/g1/meshes/right_wri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
- link right_wrist_roll_link: geometry collision mesh filename=/home/z/Desktop/PBHC/description/robots/g1/meshes/right_wri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; visual mesh filename=/home/z/Desktop/PBHC/description/robots/g1/meshes/right_wri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
- link right_wrist_yaw_link: geometry collision mesh filename=/home/z/Desktop/PBHC/description/robots/g1/meshes/right_wri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; visual mesh filename=/home/z/Desktop/PBHC/description/robots/g1/meshes/right_wri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
- link torso_link: geometry collision mesh filename=/home/z/Desktop/PBHC/description/robots/g1/meshes/torso_lin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; visual mesh filename=/home/z/Desktop/PBHC/description/robots/g1/meshes/torso_lin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
- link waist_roll_link: geometry visual mesh filename=/home/z/Desktop/PBHC/description/robots/g1/meshes/waist_rol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
- link waist_yaw_link: geometry visual mesh filename=/home/z/Desktop/PBHC/description/robots/g1/meshes/waist_yaw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

Commit message: bug last week fixed

File: description/robots/g1/29dof_official.urdf (robot description, URDF)
Before this commit: robot g1_29dof_rev_1_0, 39 links, 38 joints
Links:
- link head_link: geometry collision mesh filename=description/robots/g1/meshes/head_link.STL; visual mesh filename=description/robots/g1/meshes/head_link.STL
- link left_ankle_pitch_link: geometry collision mesh filename=description/robots/g1/meshes/left_ankle_pitch_link.STL; visual mesh filename=description/robots/g1/meshes/left_ankle_pitch_link.STL
- link left_ankle_roll_link: geometry collision sphere radius=0.005; collision sphere radius=0.005
- link left_elbow_link: geometry collision mesh filename=description/robots/g1/meshes/left_elbow_link.STL; visual mesh filename=description/robots/g1/meshes/left_elbow_link.STL
- link left_hip_pitch_link: geometry collision mesh filename=description/robots/g1/meshes/left_hip_pitch_link.STL; visual mesh filename=description/robots/g1/meshes/left_hip_pitch_link.STL
- link left_hip_roll_link: geometry collision mesh filename=description/robots/g1/meshes/left_hip_roll_link.STL; visual mesh filename=description/robots/g1/meshes/left_hip_roll_link.STL
- link left_hip_yaw_link: geometry collision mesh filename=description/robots/g1/meshes/left_hip_yaw_link.STL; visual mesh filename=description/robots/g1/meshes/left_hip_yaw_link.STL
- link left_knee_link: geometry collision mesh filename=description/robots/g1/meshes/left_knee_link.STL; visual mesh filename=description/robots/g1/meshes/left_knee_link.STL
- link left_rubber_hand: geometry visual mesh filename=description/robots/g1/meshes/left_rubber_hand.STL
- link left_shoulder_pitch_link: geometry collision cylinder length=0.05 radius=0.03; visual mesh filename=description/robots/g1/meshes/left_shoulder_pitch_link.STL
- link left_shoulder_roll_link: geometry collision cylinder length=0.03 radius=0.03; visual mesh filename=description/robots/g1/meshes/left_shoulder_roll_link.STL
- link left_shoulder_yaw_link: geometry collision mesh filename=description/robots/g1/meshes/left_shoulder_yaw_link.STL; visual mesh filename=description/robots/g1/meshes/left_shoulder_yaw_link.STL
- link left_wrist_pitch_link: geometry collision mesh filename=description/robots/g1/meshes/left_wrist_pitch_link.STL; visual mesh filename=description/robots/g1/meshes/left_wrist_pitch_link.STL
- link left_wrist_roll_link: geometry collision mesh filename=description/robots/g1/meshes/left_wrist_roll_link.STL; visual mesh filename=description/robots/g1/meshes/left_wrist_roll_link.STL
- link left_wrist_yaw_link: geometry collision mesh filename=description/robots/g1/meshes/left_wrist_yaw_link.STL; visual mesh filename=description/robots/g1/meshes/left_wrist_yaw_link.STL
- link logo_link: geometry collision mesh filename=description/robots/g1/meshes/logo_link.STL; visual mesh filename=description/robots/g1/meshes/logo_link.STL
- link pelvis: geometry visual mesh filename=description/robots/g1/meshes/pelvis.STL
- link pelvis_contour_link: geometry collision mesh filename=description/robots/g1/meshes/pelvis_contour_link.STL; visual mesh filename=description/robots/g1/meshes/pelvis_contour_link.STL
- link right_ankle_pitch_link: geometry collision mesh filename=description/robots/g1/meshes/right_ankle_pitch_link.STL; visual mesh filename=description/robots/g1/meshes/right_ankle_pitch_link.STL
- link right_ankle_roll_link: geometry collision sphere radius=0.005; collision sphere radius=0.005
- link right_elbow_link: geometry collision mesh filename=description/robots/g1/meshes/right_elbow_link.STL; visual mesh filename=description/robots/g1/meshes/right_elbow_link.STL
- link right_hip_pitch_link: geometry collision mesh filename=description/robots/g1/meshes/right_hip_pitch_link.STL; visual mesh filename=description/robots/g1/meshes/right_hip_pitch_link.STL
- link right_hip_roll_link: geometry collision mesh filename=description/robots/g1/meshes/right_hip_roll_link.STL; visual mesh filename=description/robots/g1/meshes/right_hip_roll_link.STL
- link right_hip_yaw_link: geometry collision mesh filename=description/robots/g1/meshes/right_hip_yaw_link.STL; visual mesh filename=description/robots/g1/meshes/right_hip_yaw_link.STL
- link right_knee_link: geometry collision mesh filename=description/robots/g1/meshes/right_knee_link.STL; visual mesh filename=description/robots/g1/meshes/right_knee_link.STL
- link right_rubber_hand: geometry visual mesh filename=description/robots/g1/meshes/right_rubber_hand.STL
- link right_shoulder_pitch_link: geometry collision cylinder length=0.05 radius=0.03; visual mesh filename=description/robots/g1/meshes/right_shoulder_pitch_link.STL
- link right_shoulder_roll_link: geometry collision cylinder length=0.03 radius=0.03; visual mesh filename=description/robots/g1/meshes/right_shoulder_roll_link.STL
- link right_shoulder_yaw_link: geometry collision mesh filename=description/robots/g1/meshes/right_shoulder_yaw_link.STL; visual mesh filename=description/robots/g1/meshes/right_shoulder_yaw_link.STL
- link right_wrist_pitch_link: geometry collision mesh filename=description/robots/g1/meshes/right_wrist_pitch_link.STL; visual mesh filename=description/robots/g1/meshes/right_wrist_pitch_link.STL
- link right_wrist_roll_link: geometry collision mesh filename=description/robots/g1/meshes/right_wrist_roll_link.STL; visual mesh filename=description/robots/g1/meshes/right_wrist_roll_link.STL
- link right_wrist_yaw_link: geometry collision mesh filename=description/robots/g1/meshes/right_wrist_yaw_link.STL; visual mesh filename=description/robots/g1/meshes/right_wrist_yaw_link.STL
- link torso_link: geometry collision mesh filename=description/robots/g1/meshes/torso_link_rev_1_0.STL; visual mesh filename=description/robots/g1/meshes/torso_link_rev_1_0.STL
- link waist_roll_link: geometry visual mesh filename=description/robots/g1/meshes/waist_roll_link_rev_1_0.STL
- link waist_yaw_link: geometry visual mesh filename=description/robots/g1/meshes/waist_yaw_link_rev_1_0.STL
